File: sch.kicad_sch (KiCad schematic)
At the start: 22 parts, among them J1 USB_A, J2 USB_A, J3 USB_A, J4 USB_A, J5 SparkFun DEV-14050 (CH340G), SW1 SW_MEC_5G, U1 AMS1117-3.3, U2 CH334F, U3 ESP32-S3-WROOM-1

Commit message: feat: add fabrications files
Connections:
- no-connect marks 0 -> 39
